File: ESC_Interface/P2_DSUB15_Female/P2_DSUB15_Female_V1/P2_DSUB15_Famale_V1.kicad_pcb (KiCad board)
At the start: 2 copper layers, 28 x 12 mm, 4 parts, among them J2 B4PS-VH, P2 DSUB15 Male

Commit message: Add files via upload
Parts:
- moved D1 1.73 mm to (141.7, 59.3)
- moved JP1 1.51 mm to (139.5, 59.3)
- moved J2 1.50 mm to (135.6, 59.4)
Routing:
- net /KEY+: track 11.9 -> 10.9 mm
- net /LED-: track 7.87 -> 6.98 mm
- net /KEY-: track 8.30 -> 7.48 mm
- net /GND_EXT: track 8.07 -> 7.45 mm
- net /+12V_EXT: track 7.54 -> 8.17 mm
- net /LED+: track 11.6 -> 11.0 mm
Other:
- board size 28 x 12 mm -> 24.6 x 12 mm
Changed lines of the file:
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@@
   (net 18 "unconnected-(J2-Pin_4-Pad4)")
   (footprint "Connector_JST:JST_VH_B4PS-VH_1x04_P3.96mm_Horizontal" (layer "F.Cu")
-    (at 137.14 59.4 180)
+    (at 135.64 59.4 180)
     (descr "JST VH series connector, B4PS-VH (http://www.jst-mfg.com/product/pdf/eng/eVH.pdf), generated with kicad-footprint-generator")
     (tags "connector JST VH top entry")
@@
   )
   (footprint "LED_SMD:LED_0603_1608Metric" (layer "F.Cu")
-    (at 143.4 59 90)
+    (at 141.7 59.3 90)
     (descr "LED SMD 0603 (1608 Metric), square (rectangular) end terminal, IPC_7351 nominal, (Body size source: http://www.tortai-tech.com/upload/download/2011102023233369053.pdf), generated with kicad-footprint-generator")
     (tags "LED")
@@
   )
   (footprint "Jumper:SolderJumper-2_P1.3mm_Open_TrianglePad1.0x1.5mm" (layer "F.Cu")
-    (at 141 59.1 -90)
+    (at 139.5 59.3 -90)
     (descr "SMD Solder Jumper, 1x1.5mm Triangular Pads, 0.3mm gap, open")
     (tags "solder jumper open")
@@
     )
   )
-  (gr_rect (start 117.2 56.7) (end 145.2 68.7)
+  (gr_rect (start 118.7 56.7) (end 143.3 68.7)
     (stroke (width 0.05) (type default)) (fill none) (layer "Edge.Cuts"))
   (gr_text "TACTOR+" (at 127.4 63.2 90) (layer "B.SilkS")
@@
     (effects (font (size 0.8 0.8) (thickness 0.15) bold) (justify left bottom mirror))
   )
-  (gr_text "P2_V1\n240621" (at 117.9 60.4) (layer "F.SilkS")
+  (gr_text "P2_V1\n240621" (at 121.3 61.3 90) (layer "F.SilkS")
     (effects (font (size 0.8 0.8) (thickness 0.15) bold) (justify left bottom))
   )
@@
     (effects (font (size 0.8 0.8) (thickness 0.15) bold) (justify left bottom))
   )
-  (gr_text "NC" (at 129.2 61.65) (layer "F.SilkS")
+  (gr_text "NC" (at 127.6 61.5) (layer "F.SilkS")
     (effects (font (size 0.8 0.8) (thickness 0.15)))
   )
@@
     (effects (font (size 0.8 0.8) (thickness 0.15) bold) (justify left bottom))
   )
-  (gr_text "NC" (at 125.3 61.6) (layer "F.SilkS")
+  (gr_text "NC" (at 123.5 61.5) (layer "F.SilkS")
     (effects (font (size 0.8 0.8) (thickness 0.15)))
   )
-  (gr_text "GND" (at 137.2 61.8) (layer "F.SilkS")
+  (gr_text "GND" (at 135.9 61.7) (layer "F.SilkS")
     (effects (font (size 0.8 0.8) (thickness 0.15)))
   )
@@
     (effects (font (size 0.8 0.8) (thickness 0.15) bold) (justify left bottom))
   )
-  (gr_text "+12V" (at 132.9 61.6) (layer "F.SilkS")
+  (gr_text "+12V" (at 131.6 61.4) (layer "F.SilkS")
     (effects (font (size 0.8 0.8) (thickness 0.15)))
   )
-  (gr_text "EMERG_IN-" (at 134.3 68.6 90) (layer "F.SilkS")
-    (effects (font (size 0.8 0.8) (thickness 0.15) bold) (justify left bottom))
-  )
-  (segment (start 135.215 61.325) (end 137.14 59.4) (width 1) (layer "F.Cu") (net 6))
-  (segment (start 135.215 66.675) (end 135.215 61.325) (width 1) (layer "F.Cu") (net 6))
-  (segment (start 137.985 66.675) (end 137.985 62.84) (width 0.5) (layer "F.Cu") (net 7))
+  (gr_text "EMERG_IN-" (at 134.3 68.7 90) (layer "F.SilkS")
+    (effects (font (size 0.8 0.8) (thickness 0.15) bold) (justify left bottom))
+  )
+  (segment (start 135.215 59.825) (end 135.64 59.4) (width 1) (layer "F.Cu") (net 6))
+  (segment (start 135.215 66.675) (end 135.215 59.825) (width 1) (layer "F.Cu") (net 6))
+  (segment (start 137.985 63.015) (end 139.5 61.5) (width 0.5) (layer "F.Cu") (net 7))
   (segment (start 137.985 66.675) (end 138.125 66.535) (width 0.5) (layer "F.Cu") (net 7))
-  (segment (start 137.985 62.84) (end 141 59.825) (width 0.5) (layer "F.Cu") (net 7))
-  (segment (start 140.755 62.545) (end 143.4 59.9) (width 0.5) (layer "F.Cu") (net 8))
-  (segment (start 140.755 66.675) (end 140.755 62.545) (width 0.5) (layer "F.Cu") (net 8))
-  (segment (start 133.83 66.675) (end 133.83 60.05) (width 1) (layer "B.Cu") (net 13))
-  (segment (start 133.83 60.05) (end 133.18 59.4) (width 1) (layer "B.Cu") (net 13))
-  (segment (start 141 58.375) (end 141 57.5) (width 0.5) (layer "F.Cu") (net 14))
-  (via (at 141 57.5) (size 0.6) (drill 0.3) (layers "F.Cu" "B.Cu") (net 14))
-  (segment (start 141 57.5) (end 141 60) (width 0.5) (layer "B.Cu") (net 14))
-  (segment (start 141 60) (end 136.6 64.4) (width 0.5) (layer "B.Cu") (net 14))
+  (segment (start 137.985 66.675) (end 137.985 63.015) (width 0.5) (layer "F.Cu") (net 7))
+  (segment (start 139.5 61.5) (end 139.5 60.025) (width 0.5) (layer "F.Cu") (net 7))
+  (segment (start 140.755 62.345) (end 141.7 61.4) (width 0.5) (layer "F.Cu") (net 8))
+  (segment (start 140.755 66.675) (end 140.755 62.345) (width 0.5) (layer "F.Cu") (net 8))
+  (segment (start 141.7 61.4) (end 141.7 60.0875) (width 0.5) (layer "F.Cu") (net 8))
+  (segment (start 133.83 64.73) (end 131.68 62.58) (width 1) (layer "B.Cu") (net 13))
+  (segment (start 133.83 66.675) (end 133.83 64.73) (width 1) (layer "B.Cu") (net 13))
+  (segment (start 131.68 62.58) (end 131.68 59.4) (width 1) (layer "B.Cu") (net 13))
+  (segment (start 139.5 57.8) (end 139.5 58.575) (width 0.5) (layer "F.Cu") (net 14))
+  (via (at 139.5 57.8) (size 0.6) (drill 0.3) (layers "F.Cu" "B.Cu") (net 14))
+  (segment (start 139.5 61.5) (end 136.6 64.4) (width 0.5) (layer "B.Cu") (net 14))
   (segment (start 136.6 64.4) (end 136.6 66.675) (width 0.5) (layer "B.Cu") (net 14))
-  (segment (start 143.4 57.5) (end 143.4 58.2125) (width 0.5) (layer "F.Cu") (net 15))
-  (via (at 143.4 57.5) (size 0.6) (drill 0.3) (layers "F.Cu" "B.Cu") (net 15))
+  (segment (start 139.5 57.8) (end 139.5 61.5) (width 0.5) (layer "B.Cu") (net 14))
+  (segment (start 141.7 58.5125) (end 141.7 57.6) (width 0.5) (layer "F.Cu") (net 15))
+  (via (at 141.7 57.6) (size 0.6) (drill 0.3) (layers "F.Cu" "B.Cu") (net 15))
   (segment (start 139.37 63.83) (end 139.37 66.675) (width 0.5) (layer "B.Cu") (net 15))
-  (segment (start 143.4 59.8) (end 139.37 63.83) (width 0.5) (layer "B.Cu") (net 15))
-  (segment (start 143.4 57.5) (end 143.4 59.8) (width 0.5) (layer "B.Cu") (net 15))
+  (segment (start 141.7 57.6) (end 141.7 61.5) (width 0.5) (layer "B.Cu") (net 15))
+  (segment (start 141.7 61.5) (end 139.37 63.83) (width 0.5) (layer "B.Cu") (net 15))
 )
