File: ESC_Interface/P2_DSUB15_Female/P2_DSUB15_Female_V1/P2_DSUB15_Famale_V1.kicad_sch (KiCad schematic)
At the start: 4 parts, among them J2 B4PS-VH, P2 DSUB15 Male

Commit message: Add files via upload
Parts:
- P2: value DSUB15 Male -> DSUB15 Female
