File: ESC_Interface/P3_DSUB15_Male/P3_DSUB15_Male_V1/P3_DSUB15_Male_V1.kicad_pcb (KiCad board)
At the start: 2 copper layers, 27.1 x 12 mm, 3 parts, among them J1 B2PS-VH, J2 4P_Header, P3 DA15

Commit message: Add files via upload
Parts:
- renumbered J2 to J3, J1 to J4
Other:
- board size 27.1 x 12 mm -> 24.5 x 12 mm
Changed lines of the file:
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@@
     (property "ki_keywords" "connector")
     (attr through_hole)
-    (fp_text reference "J2" (at -0.3 9.78) (layer "F.SilkS")
+    (fp_text reference "J3" (at 3.5 3.48) (layer "F.SilkS")
         (effects (font (size 0.8 0.8) (thickness 0.15)))
     )
@@
     (property "ki_keywords" "connector")
     (attr through_hole)
-    (fp_text reference "J1" (at -3.34 0) (layer "F.SilkS")
+    (fp_text reference "J4" (at -3.34 0) (layer "F.SilkS")
         (effects (font (size 0.8 0.8) (thickness 0.15)))
     )
@@
     )
   )
-  (gr_rect (start 131.2 70.5) (end 158.3 82.5)
+  (gr_rect (start 132.5 70.5) (end 157 82.5)
     (stroke (width 0.05) (type default)) (fill none) (layer "Edge.Cuts"))
   (gr_text "CAN_L" (at 143.9 78.7 90) (layer "B.SilkS")
