File: ESC_Interface/P3_DSUB15_Male/P3_DSUB15_Male_V1/P3_DSUB15_Male_V1.kicad_sch (KiCad schematic)
At the start: 3 parts, among them J1 B2PS-VH, J2 4P_Header, P3 DA15

Commit message: Add files via upload
Parts:
- renumbered J2 to J3, J1 to J4
Changed lines of the file:
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@@
   (symbol (lib_id "Connector:Conn_01x04_Pin") (at 158.75 82.55 180) (unit 1)
     (in_bom yes) (on_board yes) (dnp no)
-    (property "Reference" "J2" (at 163.83 83.82 0)
+    (property "Reference" "J3" (at 163.83 83.82 0)
       (effects (font (size 1.27 1.27)))
     )
@@
       (project "P3_DSUB15_Male_V1"
         (path "/982f3ef8-0476-4937-946f-4c922d7f21ea"
-          (reference "J2") (unit 1)
+          (reference "J3") (unit 1)
         )
       )
@@
   (symbol (lib_id "Connector:Conn_01x02_Pin") (at 158.75 92.71 180) (unit 1)
     (in_bom yes) (on_board yes) (dnp no)
-    (property "Reference" "J1" (at 160.02 92.71 0)
+    (property "Reference" "J4" (at 160.02 92.71 0)
       (effects (font (size 1.27 1.27)) (justify right))
     )
@@
       (project "P3_DSUB15_Male_V1"
         (path "/982f3ef8-0476-4937-946f-4c922d7f21ea"
-          (reference "J1") (unit 1)
+          (reference "J4") (unit 1)
         )
       )

Commit message: Add files via upload
Parts:
- P3: value DA15 -> DSUB15 Female; Link (none) -> https://www.digikey.jp/en/products/detail/amphenol-cs-fci/D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; MPN (none) -> DA15P064HTXLF
