File: ESC_Interface/P4_DSUB9_Male/P4_DSUB9_Male_V0/P4_DSUB9_Male_V0.kicad_sch (KiCad schematic)
At the start: 2 parts, among them J2 Conn_2Rows-09Pins, P4 DSUB9 Male

Commit message: Add files via upload
Parts:
- renumbered J2 to J5
Changed lines of the file:
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@@
   (symbol (lib_id "Connector_Generic:Conn_2Rows-09Pins_DSUB") (at 158.75 76.2 0) (unit 1)
     (in_bom yes) (on_board yes) (dnp no)
-    (property "Reference" "J2" (at 158.75 64.77 0)
+    (property "Reference" "J5" (at 158.75 64.77 0)
       (effects (font (size 1.27 1.27)))
     )
@@
     (pin "10")
     (instances
-      (project "DSUB9_Male"
+      (project "P4_DSUB9_Male_V0"
         (path "/105f448c-cc44-46f7-8e84-435fd9b748b1"
-          (reference "J2") (unit 1)
+          (reference "J5") (unit 1)
         )
       )
@@
     (pin "7")
     (instances
-      (project "DSUB9_Male"
+      (project "P4_DSUB9_Male_V0"
         (path "/105f448c-cc44-46f7-8e84-435fd9b748b1"
           (reference "P4") (unit 1)
@@
     (pin "1")
     (instances
-      (project "DSUB9_Male"
+      (project "P4_DSUB9_Male_V0"
         (path "/105f448c-cc44-46f7-8e84-435fd9b748b1"
           (reference "#PWR01") (unit 1)
