File: ESC_Interface/P4_DSUB9_Male/P4_DSUB9_Male_V0/P4_DSUB9_Male_V0.kicad_pcb (KiCad board)
At the start: 2 copper layers, 20 x 12 mm, 3 parts, among them J2 Conn_2Rows-09Pins, P4 DE9_Receptacle_MountingHoles

Commit message: Add files via upload
Parts:
- removed REF**: JST_VH_B2PS-VH_1x02_P3.96mm_Horizontal, Connector_JST:JST_VH_B2PS-VH_1x02_P3.96mm_Horizontal
- renumbered J2 to J5
Other:
- board size 20 x 12 mm -> 16.1 x 12 mm
Changed lines of the file:
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@@
   (net 10 "/TEMP+")
   (net 11 "unconnected-(P4-PAD-Pad0)")
-  (footprint "Connector_JST:JST_VH_B2PS-VH_1x02_P3.96mm_Horizontal" (layer "F.Cu")
-    (at 81 65.2)
-    (descr "JST VH series connector, B2PS-VH (http://www.jst-mfg.com/product/pdf/eng/eVH.pdf), generated with kicad-footprint-generator")
-    (tags "connector JST VH top entry")
-    (attr through_hole)
-    (fp_text reference "REF**" (at 1.98 -2.55) (layer "F.SilkS")
-        (effects (font (size 1 1) (thickness 0.15)))
-    )
-    (fp_text value "JST_VH_B2PS-VH_1x02_P3.96mm_Horizontal" (at 1.98 16.1) (layer "F.Fab")
-        (effects (font (size 1 1) (thickness 0.15)))
-    )
-    (fp_text user "${REFERENCE}" (at 1.98 9.45) (layer "F.Fab")
-        (effects (font (size 1 1) (thickness 0.15)))
-    )
-    (fp_line (start -2.06 3.89) (end 6.02 3.89)
-      (stroke (width 0.12) (type solid)) (layer "F.SilkS"))
-    (fp_line (start -2.06 7.31) (end -2.06 3.89)
-      (stroke (width 0.12) (type solid)) (layer "F.SilkS"))
-    (fp_line (start -1.61 -1.61) (end -1.61 0)
-      (stroke (width 0.12) (type solid)) (layer "F.SilkS"))
-    (fp_line (start -1.01 7.31) (end -2.06 7.31)
-      (stroke (width 0.12) (type solid)) (layer "F.SilkS"))
-    (fp_line (start -1.01 13.51) (end -1.01 7.31)
-      (stroke (width 0.12) (type solid)) (layer "F.SilkS"))
-    (fp_line (start -0.82 13.51) (end -0.82 15.01)
-      (stroke (width 0.12) (type solid)) (layer "F.SilkS"))
-    (fp_line (start -0.82 15.01) (end 0.82 15.01)
-      (stroke (width 0.12) (type solid)) (layer "F.SilkS"))
-    (fp_line (start 0 -1.61) (end -1.61 -1.61)
-      (stroke (width 0.12) (type solid)) (layer "F.SilkS"))
-    (fp_line (start 0.82 15.01) (end 0.82 13.51)
-      (stroke (width 0.12) (type solid)) (layer "F.SilkS"))
-    (fp_line (start 3.14 13.51) (end 3.14 15.01)
-      (stroke (width 0.12) (type solid)) (layer "F.SilkS"))
-    (fp_line (start 3.14 15.01) (end 4.78 15.01)
-      (stroke (width 0.12) (type solid)) (layer "F.SilkS"))
-    (fp_line (start 4.78 15.01) (end 4.78 13.51)
-      (stroke (width 0.12) (type solid)) (layer "F.SilkS"))
-    (fp_line (start 4.97 7.31) (end 4.97 13.51)
-      (stroke (width 0.12) (type solid)) (layer "F.SilkS"))
-    (fp_line (start 4.97 13.51) (end -1.01 13.51)
-      (stroke (width 0.12) (type solid)) (layer "F.SilkS"))
-    (fp_line (start 6.02 3.89) (end 6.02 7.31)
-      (stroke (width 0.12) (type solid)) (layer "F.SilkS"))
-    (fp_line (start 6.02 7.31) (end 4.97 7.31)
-      (stroke (width 0.12) (type solid)) (layer "F.SilkS"))
-    (fp_line (start -2.45 -1.85) (end -2.45 15.4)
-      (stroke (width 0.05) (type solid)) (layer "F.CrtYd"))
-    (fp_line (start -2.45 15.4) (end 6.41 15.4)
-      (stroke (width 0.05) (type solid)) (layer "F.CrtYd"))
-    (fp_line (start 6.41 -1.85) (end -2.45 -1.85)
-      (stroke (width 0.05) (type solid)) (layer "F.CrtYd"))
-    (fp_line (start 6.41 15.4) (end 6.41 -1.85)
-      (stroke (width 0.05) (type solid)) (layer "F.CrtYd"))
-    (fp_line (start -1.95 4) (end -0.9 4)
-      (stroke (width 0.1) (type solid)) (layer "F.Fab"))
-    (fp_line (start -1.95 7.2) (end -1.95 4)
-      (stroke (width 0.1) (type solid)) (layer "F.Fab"))
-    (fp_line (start -0.9 4) (end -0.9 13.4)
-      (stroke (width 0.1) (type solid)) (layer "F.Fab"))
-    (fp_line (start -0.9 7.2) (end -1.95 7.2)
-      (stroke (width 0.1) (type solid)) (layer "F.Fab"))
-    (fp_line (start -0.9 13.4) (end 4.86 13.4)
-      (stroke (width 0.1) (type solid)) (layer "F.Fab"))
-    (fp_line (start -0.8 4) (end 0 4.8)
-      (stroke (width 0.1) (type solid)) (layer "F.Fab"))
-    (fp_line (start -0.7 0) (end 0.7 0)
-      (stroke (width 0.1) (type solid)) (layer "F.Fab"))
-    (fp_line (start -0.7 4) (end -0.7 0)
-      (stroke (width 0.1) (type solid)) (layer "F.Fab"))
-    (fp_line (start -0.7 13.4) (end -0.7 14.9)
-      (stroke (width 0.1) (type solid)) (layer "F.Fab"))
-    (fp_line (start -0.7 14.9) (end 0.7 14.9)
-      (stroke (width 0.1) (type solid)) (layer "F.Fab"))
-    (fp_line (start 0 4.8) (end 0.8 4)
-      (stroke (width 0.1) (type solid)) (layer "F.Fab"))
-    (fp_line (start 0.7 0) (end 0.7 4)
-      (stroke (width 0.1) (type solid)) (layer "F.Fab"))
-    (fp_line (start 0.7 14.9) (end 0.7 13.4)
-      (stroke (width 0.1) (type solid)) (layer "F.Fab"))
-    (fp_line (start 3.26 0) (end 4.66 0)
-      (stroke (width 0.1) (type solid)) (layer "F.Fab"))
-    (fp_line (start 3.26 4) (end 3.26 0)
-      (stroke (width 0.1) (type solid)) (layer "F.Fab"))
-    (fp_line (start 3.26 13.4) (end 3.26 14.9)
-      (stroke (width 0.1) (type solid)) (layer "F.Fab"))
-    (fp_line (start 3.26 14.9) (end 4.66 14.9)
-      (stroke (width 0.1) (type solid)) (layer "F.Fab"))
-    (fp_line (start 4.66 0) (end 4.66 4)
-      (stroke (width 0.1) (type solid)) (layer "F.Fab"))
-    (fp_line (start 4.66 14.9) (end 4.66 13.4)
-      (stroke (width 0.1) (type solid)) (layer "F.Fab"))
-    (fp_line (start 4.86 4) (end -0.9 4)
-      (stroke (width 0.1) (type solid)) (layer "F.Fab"))
-    (fp_line (start 4.86 4) (end 5.91 4)
-      (stroke (width 0.1) (type solid)) (layer "F.Fab"))
-    (fp_line (start 4.86 13.4) (end 4.86 4)
-      (stroke (width 0.1) (type solid)) (layer "F.Fab"))
-    (fp_line (start 5.91 4) (end 5.91 7.2)
-      (stroke (width 0.1) (type solid)) (layer "F.Fab"))
-    (fp_line (start 5.91 7.2) (end 4.86 7.2)
-      (stroke (width 0.1) (type solid)) (layer "F.Fab"))
-    (pad "1" thru_hole roundrect (at 0 0) (size 2.7 2.7) (drill 1.7) (layers "*.Cu" "*.Mask") (roundrect_rratio 0.092593))
-    (pad "2" thru_hole circle (at 3.96 0) (size 2.7 2.7) (drill 1.7) (layers "*.Cu" "*.Mask"))
-    (model "${KICAD6_3DMODEL_DIR}/Connector_JST.3dshapes/JST_VH_B2PS-VH_1x02_P3.96mm_Horizontal.wrl"
-      (offset (xyz 0 0 0))
-      (scale (xyz 1 1 1))
-      (rotate (xyz 0 0 0))
-    )
-  )
   (footprint "Connector_Dsub:DSUB-9_Male_Calendar_P2.77x2.84mm_MountingHoles3.1mm_24.99" (layer "F.Cu")
     (at 138.4 87)
@@
     (property "ki_keywords" "connector receptacle female D-SUB DB9")
     (attr through_hole)
-    (fp_text reference "P4" (at -8.1 -13.5) (layer "F.SilkS")
+    (fp_text reference "P4" (at -7.1 -13.6) (layer "F.SilkS")
         (effects (font (size 0.8 0.8) (thickness 0.15)))
     )
@@
       (net 10 "/TEMP+") (pinfunction "9") (pintype "passive"))
     (model "${KICAD7_3DMODEL_DIR}/Connector_Dsub.3dshapes/DSUB-9-Male_DE09P065HTXLF.STEP"
-      (offset (xyz 0.05 0.51 -0.85))
+      (offset (xyz 0.05 -9.99 9.15))
       (scale (xyz 1 1 1))
       (rotate (xyz -90 0 0))
+    )
+    (model "C:/Users/Administrator/Desktop/977-009-010R031.step/977-009-010R031.STEP"
+      (offset (xyz 0 -8.5 1.5))
+      (scale (xyz 1 1 1))
+      (rotate (xyz 0 0 0))
     )
   )
@@
     (property "ki_keywords" "connector")
     (attr through_hole)
-    (fp_text reference "J2" (at -0.65 -3.25 180) (layer "F.SilkS")
+    (fp_text reference "J5" (at -0.05 -2.25 180) (layer "F.SilkS")
         (effects (font (size 0.8 0.8) (thickness 0.15)))
     )
@@
   (gr_line (start 131.8 71.3) (end 131 70.9)
     (stroke (width 0.1) (type default)) (layer "B.SilkS"))
-  (gr_line (start 129.9 71.3) (end 131.8 71.3)
-    (stroke (width 0.1) (type default)) (layer "B.SilkS"))
-  (gr_line (start 132.1 75.3) (end 129.9 73)
-    (stroke (width 0.1) (type default)) (layer "B.SilkS"))
-  (gr_line (start 129.9 71.3) (end 129.9 73)
-    (stroke (width 0.1) (type default)) (layer "B.SilkS"))
-  (gr_rect (start 128.4 69.5) (end 148.4 81.5)
+  (gr_line (start 130.8 71.3) (end 131.8 71.3)
+    (stroke (width 0.1) (type default)) (layer "B.SilkS"))
+  (gr_line (start 132.1 75.3) (end 130.8 73)
+    (stroke (width 0.1) (type default)) (layer "B.SilkS"))
+  (gr_line (start 130.8 71.3) (end 130.8 73)
+    (stroke (width 0.1) (type default)) (layer "B.SilkS"))
+  (gr_rect (start 130.4 69.5) (end 146.5 81.5)
     (stroke (width 0.05) (type default)) (fill none) (layer "Edge.Cuts"))
   (gr_text "SEN_B" (at 143.6 81.4 270) (layer "B.SilkS")
@@
     (effects (font (size 0.8 0.8) (thickness 0.15) bold) (justify left bottom))
   )
-  (gr_text "240621" (at 147.1 74.2 90) (layer "F.SilkS")
-    (effects (font (size 0.8 0.8) (thickness 0.15) bold) (justify left bottom))
-  )
+  (gr_text "240621" (at 146.1 74.2 90) (layer "F.SilkS")
+    (effects (font (size 0.8 0.8) (thickness 0.15) bold) (justify left bottom))
+  )

Commit message: Add files via upload
Parts:
- moved J5 1.81 mm to (133.4, 73.2)
Routing:
- net /SEN_A: track 5.78 -> 3.94 mm
- net /GEN_SEN: track 5.68 -> 3.85 mm
- net /SEN_C: track 5.88 -> 4.04 mm
- net /SEN_B: track 8.88 -> 7.07 mm
- net +12V: track 8.73 -> 6.95 mm
- net /SHIELD: track 5.71 -> 3.93 mm
- net /TEMP+: track 8.82 -> 7.04 mm
- net /TEMP-: track 5.80 -> 4.02 mm
Other:
- board size 16.1 x 12 mm -> 16.1 x 10 mm
