File: ESC_Interface/ESC_Interface_All/ESC_Interface_All.kicad_pcb (KiCad board)
At the start: 2 copper layers, 115.8 x 12 mm, 11 parts, among them J1 Conn_01x03_Pin, J2 B4PS-VH, J3 4P_Header, J4 B2PS-VH, J5 Conn_2Rows-09Pins, P1 DB25_Male, P2 DSUB15 Male, P3 DA15, P4 DE9_Receptacle_MountingHoles

Commit message: Add files via upload
Parts:
- P4: value DE9_Receptacle_MountingHoles -> DSUB9 Male
- moved JP1 2.27 mm to (126.0, 89.6)
- moved D1 2.21 mm to (128.1, 89.4)
- moved J2 1.77 mm to (122.1, 89.4)
- moved J3 1.76 mm to (143.9, 88.8)
- moved J1 1.63 mm to (86.4, 90.1)
- moved J4 1.61 mm to (152.2, 89.2)
- moved J5 1.53 mm to (165.7, 88.5)
Connections:
- D1 pad 1: (no net) -> /LED-
- D1 pad 2: (no net) -> /LED+
- J1 pad 1: (no net) -> /PWM1+
- J1 pad 2: (no net) -> /PWM-
- J1 pad 3: (no net) -> /PWM-
- J2 pad 1: (no net) -> /GND_EXT
- J2 pad 2: (no net) -> /+12V_EXT
- J2 pad 3: (no net) -> unconnected-(J2-Pin_3-Pad3)
- J2 pad 4: (no net) -> unconnected-(J2-Pin_4-Pad4)
- J3 pad 1: (no net) -> /TX_USB
- J3 pad 2: (no net) -> /RX_USB
- J3 pad 3: (no net) -> /3.3V_OUT
- J3 pad 4: (no net) -> /GND_USB
- J4 pad 1: (no net) -> /CAN_H
- J4 pad 2: (no net) -> /CAL_L
- J5 pad 1: (no net) -> /SEN_C
- J5 pad 10: (no net) -> unconnected-(J5-Pin_10-Pad10)
- J5 pad 2: (no net) -> /SEN_A
- J5 pad 3: (no net) -> /GEN_SEN
- J5 pad 4: (no net) -> /SHIELD
- J5 pad 5: (no net) -> /TEMP-
- J5 pad 6: (no net) -> /SEN_B
- J5 pad 7: (no net) -> /ABS_POS
- J5 pad 8: (no net) -> +12V
- J5 pad 9: (no net) -> /TEMP+
- JP1 pad 1: (no net) -> /KEY+
- JP1 pad 2: (no net) -> /KEY-
- P1 pad 0: (no net) -> unconnected-(P1-PAD-Pad0)
- P1 pad 1: (no net) -> /OUT_32
- P1 pad 10: (no net) -> /INA_26+
- P1 pad 11: (no net) -> /INA_27+
- P1 pad 12: (no net) -> /(AUX)PWM2+
- P1 pad 13: (no net) -> /GND1
- P1 pad 14: (no net) -> /TX(OUT_31)
- P1 pad 15: (no net) -> /N.C.
- P1 pad 16: (no net) -> /IN_21+
- P1 pad 17: (no net) -> /INA_22+
- P1 pad 18: (no net) -> /IN_20+
- P1 pad 19: (no net) -> /+5V_LED
- P1 pad 2: (no net) -> /(IN_31)_RX
- P1 pad 20: (no net) -> /OUT_24
- P1 pad 21: (no net) -> /SHIELD_POT
- P1 pad 22: (no net) -> /(AUX)INA_25+
- P1 pad 23: (no net) -> /INA_U-
- P1 pad 24: (no net) -> /PWM1+
- P1 pad 25: (no net) -> /PWM-
- P1 pad 3: (no net) -> /GND1(RX/TX&OUT_32)
- P1 pad 4: (no net) -> /IN_21-
- P1 pad 5: (no net) -> /INA_22-
- P1 pad 6: (no net) -> /IN_20-
- P1 pad 7: (no net) -> /OUT_23
- P1 pad 8: (no net) -> /GND(OUT_23&24)
- P1 pad 9: (no net) -> /INA_U+
- P2 pad 0: (no net) -> unconnected-(P2-PAD-Pad0)
- P2 pad 1: (no net) -> /(GND_EXT)
- P2 pad 10: (no net) -> /CONTACTOR-
- P2 pad 11: (no net) -> /CONTACTOR+
- P2 pad 12: (no net) -> /ENERG_U+
- P2 pad 13: (no net) -> /+12V_EXT
- P2 pad 14: (no net) -> /KEY+
- P2 pad 15: (no net) -> /LED+
- P2 pad 2: (no net) -> /RELAY-
- P2 pad 3: (no net) -> /RELAY+
- P2 pad 4: (no net) -> /EMERG_IN+
- P2 pad 5: (no net) -> /EMERG_IN-
- P2 pad 6: (no net) -> /GND_EXT
- P2 pad 7: (no net) -> /KEY-
- P2 pad 8: (no net) -> /LED-
- P2 pad 9: (no net) -> /EMERG_U-
- P3 pad 0: (no net) -> unconnected-(P3-PAD-Pad0)
- P3 pad 1: (no net) -> /GND_COM1
- P3 pad 10: (no net) -> /3.3V_OUT
- P3 pad 11: (no net) -> /TX_USB
- P3 pad 12: (no net) -> /CAL_L
- P3 pad 13: (no net) -> /Z120_C
- P3 pad 14: (no net) -> /RS485_B-
- P3 pad 15: (no net) -> /Z120_R
- P3 pad 2: (no net) -> /GND_USB
- P3 pad 3: (no net) -> /RX_USB
- P3 pad 4: (no net) -> /NC0
- P3 pad 5: (no net) -> /CAN_H
- P3 pad 6: (no net) -> /GND_COM3
- P3 pad 7: (no net) -> /RS485_A+
- P3 pad 8: (no net) -> /NC1
- P3 pad 9: (no net) -> /GND_COM2
- P4 pad 0: (no net) -> unconnected-(P4-PAD-Pad0)
- P4 pad 1: (no net) -> /SEN_C
- P4 pad 2: (no net) -> /SEN_A
- P4 pad 3: (no net) -> /GEN_SEN
- P4 pad 4: (no net) -> /SHIELD
- P4 pad 5: (no net) -> /TEMP-
- P4 pad 6: (no net) -> /SEN_B
- P4 pad 7: (no net) -> /ABS_POS
- P4 pad 8: (no net) -> +12V
- P4 pad 9: (no net) -> /TEMP+
Routing:
- net (no net): track 204.4 -> 0.00 mm, vias 2 -> 0
- net /PWM-: track 0.00 -> 23.3 mm
- net /PWM1+: track 0.00 -> 10.9 mm
- net /KEY+: track 0.00 -> 9.40 mm, vias 0 -> 1
- net /LED+: track 0.00 -> 8.83 mm, vias 0 -> 1
- net /CAN_H: track 0.00 -> 7.68 mm
- net /SEN_B: track 0.00 -> 7.35 mm
- net /TEMP+: track 0.00 -> 7.30 mm
- net /ABS_POS: track 0.00 -> 7.26 mm
- net +12V: track 0.00 -> 7.20 mm
- net /GND_USB: track 0.00 -> 7.19 mm
- net /3.3V_OUT: track 0.00 -> 6.99 mm
- net /CAL_L: track 0.00 -> 6.62 mm
- net /RX_USB: track 0.00 -> 6.51 mm
- net /+12V_EXT: track 0.00 -> 6.49 mm
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Other:
- board size 115.8 x 12 mm -> 114.7 x 10 mm
- board text added: "<-V-cut"

Commit message: Add files via upload
Other:
- board size 114.7 x 10 mm -> 119.9 x 23 mm
Changed lines of the file:
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@@
     )
   )
-  (gr_rect (start 106 87) (end 129.5 97)
+  (gr_rect (start 106 74) (end 129.5 97)
     (stroke (width 0.05) (type default)) (fill none) (layer "B.SilkS"))
   (gr_line (start 164.35 87.55) (end 163.55 87.15)
@@
   (gr_line (start 163.25 87.55) (end 164.35 87.55)
     (stroke (width 0.1) (type default)) (layer "B.SilkS"))
-  (gr_rect (start 134.6 87) (end 158.1 97)
+  (gr_rect (start 134.6 73.9) (end 158.1 97)
     (stroke (width 0.05) (type default)) (fill none) (layer "B.SilkS"))
   (gr_line (start 165.1 92.9) (end 163.25 89.2625)
     (stroke (width 0.1) (type default)) (layer "B.SilkS"))
-  (gr_rect (start 63.5 87) (end 100.9 97)
+  (gr_rect (start 63.5 73.9) (end 100.9 97)
     (stroke (width 0.05) (type default)) (fill none) (layer "B.SilkS"))
   (gr_rect (start 163.1 87) (end 178.2 97)
@@
   (gr_line (start 177.05 93.8) (end 177.05 94.75)
     (stroke (width 0.1) (type default)) (layer "F.SilkS"))
-  (gr_line (start 163.1 87) (end 163.1 97)
+  (gr_line (start 160.7 74) (end 160.7 97)
     (stroke (width 0.2) (type default)) (layer "Edge.Cuts"))
-  (gr_line (start 129.5 87) (end 129.5 97)
+  (gr_rect (start 60.9 74) (end 180.8 97)
+    (stroke (width 0.05) (type default)) (fill none) (layer "Edge.Cuts"))
+  (gr_line (start 132 74) (end 132 97)
     (stroke (width 0.2) (type default)) (layer "Edge.Cuts"))
-  (gr_line (start 100.9 87) (end 100.9 97)
-    (stroke (width 0.2) (type default)) (layer "Edge.Cuts"))
-  (gr_rect (start 63.5 87) (end 178.2 97)
-    (stroke (width 0.05) (type default)) (fill none) (layer "Edge.Cuts"))
-  (gr_line (start 134.65 87) (end 134.65 97.05)
-    (stroke (width 0.2) (type default)) (layer "Edge.Cuts"))
-  (gr_line (start 106 87) (end 106 97)
-    (stroke (width 0.2) (type default)) (layer "Edge.Cuts"))
-  (gr_line (start 158.1 87) (end 158.1 97)
+  (gr_line (start 103.5 74) (end 103.5 96.95)
     (stroke (width 0.2) (type default)) (layer "Edge.Cuts"))
   (gr_text "PWM1+" (at 96.35 93.25 90) (layer "B.SilkS")
@@
     (effects (font (size 0.6 0.6) (thickness 0.15)))
   )
-  (gr_text "<-V-cut" (at 158.6 85.85 90) (layer "Edge.Cuts")
-    (effects (font (size 1 1) (thickness 0.15)) (justify left bottom))
-  )
-  (gr_text "<-V-cut" (at 106.45 85.7 90) (layer "Edge.Cuts")
-    (effects (font (size 1 1) (thickness 0.15)) (justify left bottom))
-  )
-  (gr_text "<-V-cut" (at 129.95 85.75 90) (layer "Edge.Cuts")
-    (effects (font (size 1 1) (thickness 0.15)) (justify left bottom))
-  )
-  (gr_text "<-V-cut" (at 101.3 85.7 90) (layer "Edge.Cuts")
-    (effects (font (size 1 1) (thickness 0.15)) (justify left bottom))
-  )
-  (gr_text "<-V-cut" (at 163.55 85.8 90) (layer "Edge.Cuts")
-    (effects (font (size 1 1) (thickness 0.15)) (justify left bottom))
-  )
-  (gr_text "<-V-cut" (at 135.1 85.75 90) (layer "Edge.Cuts")
-    (effects (font (size 1 1) (thickness 0.15)) (justify left bottom))
-  )
+  (gr_text "<-V-cut" (at 158.5 73 90) (layer "Edge.Cuts")
+    (effects (font (size 1 1) (thickness 0.15)) (justify left bottom))
+  )
+  (gr_text "<-V-cut" (at 103.9 72.85 90) (layer "Edge.Cuts")
+    (effects (font (size 1 1) (thickness 0.15)) (justify left bottom))
+  )
+  (gr_text "<-V-cut" (at 163.45 72.95 90) (layer "Edge.Cuts")
+    (effects (font (size 1 1) (thickness 0.15)) (justify left bottom))
+  )
+  (gr_text "<-V-cut" (at 132.5 72.9 90) (layer "Edge.Cuts")
+    (effects (font (size 1 1) (thickness 0.15)) (justify left bottom))
+  )
