File: ESC_Interface/P3_DSUB15_Male/P3_DSUB15_Male_V0/P3_DSUB15_Male_V0.kicad_sch (KiCad schematic)
At the start: 2 parts, among them J1 Conn_01x15, P3 DA15

Commit message: Add files via upload
Parts:
- P3: value DA15 -> DSUB15 Male; Link (none) -> https://www.digikey.jp/en/products/detail/amphenol-cs-fci/D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; MPN (none) -> DA15P064HTXLF
